Commit message: Add files via upload
Base0 and Tool0 include in URDF file,
IKFastKinematics plugin and pilz industrial motion compatible flange and base_link

File: sr80_description/urdf/sr80_wm.urdf (robot description, URDF)
Before this commit: robot SR80, 8 links, 7 joints
Links:
- removed link L6
- added link base0
- added link flange, mass 0.001; visual box size=0.04 0.04 0.04
- added link tcp
- added link world
Joints:
- removed joint tcp_tool0
- added joint base_link-base: type fixed, parent base_link, child base0, origin xyz=0 0 0 rpy=0 0 0
- added joint fixed_joint_tcp: type fixed, parent flange, child tcp, origin xyz=0 0 0 rpy=0 0 0
- added joint flange-tool0: type fixed, parent flange, child tool0, origin xyz=0 0 0 rpy=0 0 0
- added joint world-base_link-fixed: type fixed, parent world, child base_link
- joint J6: child L6 -> flange
